File: Lil-Cheat.kicad_pcb (KiCad board)
At the start: 2 copper layers, 298.4 x 81.3 mm, 129 parts, among them J1 USB2_C_Receptacle, SW1 SW_Push, U1 ATmega32U2-AU, U2 SRV05-4, Y1 16MHz

Commit message: swapped to daughterboard
Parts:
- removed F1: 500mA, Fuse:Fuse_1206_3216Metric
- removed R5, R6: 5.1k, Resistor_SMD:R_0805_2012Metric
- removed U2: SRV05-4, Package_TO_SOT_SMD:SOT-23-6
- J1: value USB2_C_Receptacle -> Conn_01x04; footprint usb-type-c:Mid_Mount-USB_C -> Connector_JST:JST_SUR_SM04B-SURS-TF_1x04-1MP_P0.80mm_Horizontal
- moved R2 70.6 mm to (243.7, 91.3), turned to 90 degrees
- moved SW1 61.7 mm to (235.7, 79.9), turned to 0 degrees
- moved C4 38.2 mm to (250.0, 95.2), turned to 180 degrees
- moved R3 36.1 mm to (241.5, 91.2), turned to 270 degrees
- moved C5 34.8 mm to (250.0, 97.6), turned to 180 degrees
- moved C2 34.5 mm to (255.7, 111.7)
- moved J1 31.3 mm to (242.6, 87.1), turned to 0 degrees
- moved C3 27.8 mm to (242.9, 95.2), turned to 270 degrees
- moved C1 26.7 mm to (255.7, 104.8)
- moved R4 24.8 mm to (236.5, 113.5), turned to 90 degrees
- moved R1 24.8 mm to (245.8, 91.3), turned to 90 degrees
- moved C6 16.5 mm to (250.0, 92.9), turned to 180 degrees
- moved Y1 13.1 mm to (255.7, 108.3), turned to 270 degrees
- moved C7 11.7 mm to (250.0, 90.5), turned to 180 degrees
- moved U1 5.84 mm to (244.8, 105.9), turned to 90 degrees
Connections:
- C4 pad 2: VBUS -> +5V
- C5 pad 2: VBUS -> +5V
- C6 pad 2: VBUS -> +5V
- C7 pad 2: VBUS -> +5V
- R3 pad 1: VBUS -> +5V
- U1 pad 10: ROW2 -> COL10
- U1 pad 11: ROW3 -> COL9
- U1 pad 14: COL0 -> COL12
- U1 pad 15: COL1 -> COL8
- U1 pad 16: COL2 -> COL7
- U1 pad 17: COL3 -> COL6
- U1 pad 18: COL4 -> COL5
- U1 pad 19: COL5 -> COL4
- U1 pad 20: COL6 -> COL3
- U1 pad 21: COL7 -> ROW1
- U1 pad 22: COL12 -> COL2
- U1 pad 23: COL11 -> COL1
- U1 pad 25: COL10 -> COL0
- U1 pad 26: COL9 -> ROW0
- U1 pad 31: VBUS -> +5V
- U1 pad 32: VBUS -> +5V
- U1 pad 4: VBUS -> +5V
- U1 pad 5: COL8 -> ROW2
- U1 pad 6: COL13 -> COL14
- U1 pad 7: COL14 -> COL13
- U1 pad 8: ROW0 -> ROW3
- U1 pad 9: ROW1 -> COL11
Routing:
- net ROW3: track 0.00 -> 337.6 mm
- net GND: track 11.4 -> 57.3 mm, vias 0 -> 2
- net ROW2: track 240.2 -> 284.3 mm
- net +5V: track 0.00 -> 44.0 mm
- net ROW0: track 294.0 -> 328.4 mm, vias 0 -> 2
- net Net-(R3-Pad2): track 0.00 -> 23.2 mm
- net COL0: track 285.3 -> 304.6 mm, vias 0 -> 2
- net COL3: track 217.6 -> 236.6 mm
- net COL14: track 89.7 -> 107.6 mm
- net COL1: track 268.5 -> 285.5 mm
- net COL2: track 248.8 -> 265.3 mm
- net COL13: track 72.4 -> 87.9 mm
- net COL4: track 202.1 -> 217.5 mm
- net COL5: track 184.7 -> 198.4 mm
- net COL6: track 166.1 -> 179.3 mm
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Other:
- board size 298.4 x 81.3 mm -> 298.4 x 76.2 mm
