File: Ortho/Lil-Cheat.kicad_pcb (KiCad board)
At the start: 2 copper layers, 298.4 x 76.2 mm, 125 parts, among them J1 Conn_01x04, SW1 SW_Push, U1 ATmega32U2-AU, Y1 16MHz

Commit message: project tidy
Routing:
- net ROW3: track 336.5 -> 337.6 mm
- net +5V: track 43.2 -> 44.0 mm
